Commit message: buggy example

File: rsc/templatedTrackedRobot/trackedTemplate.urdf (robot description, URDF)
Before this commit: robot husky_robot, 27 links, 26 joints
Links:
- removed link front_left_flipper_wheel_link
- removed link front_left_flipper_wheel_link2
- removed link front_left_flipper_wheel_link3
- removed link front_left_wheel_link
- removed link front_right_flipper_wheel_link
- removed link front_right_flipper_wheel_link2
- removed link front_right_flipper_wheel_link3
- removed link front_right_wheel_link
- removed link horizontal_link
- removed link horizontal_link2
- removed link horizontal_link3
- removed link horizontal_link4
- removed link horizontal_link5
- removed link horizontal_link6
- removed link horizontal_link7
- removed link horizontal_link8
- removed link rear_left_wheel_link
- removed link rear_right_wheel_link
- removed link vertical_link
- removed link vertical_link2
- removed link vertical_link3
- removed link vertical_link4
- removed link vertical_link5
- removed link vertical_link6
- removed link vertical_link7
- removed link vertical_link8
- added link left_flipper, mass {@@rho*@@wheel_width*@@flipper_radius*@@flipper_radius*1.57}; visual cylinder length={@@wheel_width+0.02} radius={@@flipper_radius*0.3}; visual cylinder length={@@wheel_width+0.02} radius={@@flipper_radius*0.55}
- added link left_idler_link; visual cylinder length={@@wheel_width+0.02} radius={@@wheel_radius*0.55}
- added link left_sprocket_link, mass {@@rho*@@wheel_width*@@wheel_radius*@@wheel_radius*0.94}; visual box size={@@wheel_radius*1.05} {@@wheel_width+0.024} 0.03; visual cylinder length={@@wheel_width+0.02} radius={@@wheel_radius*0.55}
- added link right_flipper, mass {@@rho*@@wheel_width*@@flipper_radius*@@flipper_radius*1.57}; visual cylinder length={@@wheel_width+0.02} radius={@@flipper_radius*0.3}; visual cylinder length={@@wheel_width+0.02} radius={@@flipper_radius*0.55}
- added link right_idler_link; visual cylinder length={@@wheel_width+0.02} radius={@@wheel_radius*0.55}
- added link right_sprocket_link, mass {@@rho*@@wheel_width*@@wheel_radius*@@wheel_radius*0.94}; visual box size={@@wheel_radius*1.05} {@@wheel_width+0.024} 0.03; visual cylinder length={@@wheel_width+0.02} radius={@@wheel_radius*0.55}
- link base_link: mass {@@rho*@@base_length*@@base_width*0.2075} -> {@@rho*@@base_length*@@base_width*0.2}; geometry collision box size=@@base_length @@base_width 0.2; visual box size=@@base_length @@base_width 0.2
Joints:
- removed joint front_left_flipper_wheel
- removed joint front_left_flipper_wheel2
- removed joint front_left_flipper_wheel3
- removed joint front_left_wheel
- removed joint front_right_flipper_wheel
- removed joint front_right_flipper_wheel2
- removed joint front_right_flipper_wheel3
- removed joint front_right_wheel
- removed joint horizontal_joint
- removed joint horizontal_joint2
- removed joint horizontal_joint3
- removed joint horizontal_joint4
- removed joint horizontal_joint5
- removed joint horizontal_joint6
- removed joint horizontal_joint7
- removed joint horizontal_joint8
- removed joint rear_left_wheel
- removed joint rear_right_wheel
- removed joint vertical_joint
- removed joint vertical_joint2
- removed joint vertical_joint3
- removed joint vertical_joint4
- removed joint vertical_joint5
- removed joint vertical_joint6
- removed joint vertical_joint7
- removed joint vertical_joint8
- added joint left_flipper_joint: type continuous, parent base_link, child left_flipper, origin xyz={@@base_length*0.5} @@track_y_offset 0, axis 0 1 0
- added joint left_idler: type fixed, parent base_link, child left_idler_link, origin xyz=-{@@base_length*0.5} @@wheel_y_offset 0
- added joint left_sprocket: type continuous, parent base_link, child left_sprocket_link, origin xyz={@@base_length*0.5} @@wheel_y_offset 0, axis 0 1 0
- added joint right_flipper_joint: type continuous, parent base_link, child right_flipper, origin xyz={@@base_length*0.5} -@@track_y_offset 0, axis 0 1 0
- added joint right_idler: type fixed, parent base_link, child right_idler_link, origin xyz=-{@@base_length*0.5} -@@wheel_y_offset 0
- added joint right_sprocket: type continuous, parent base_link, child right_sprocket_link, origin xyz={@@base_length*0.5} -@@wheel_y_offset 0, axis 0 1 0
